File: pcb/modular.sch (KiCad schematic (older format))
At the start: 41 parts, among them J1 USB_OTG, J2 OUTPUT1, J3 OUTPUT2, J4 GPIO, J5 INPUT1, J6 INPUT2, J7 BOOT, SW1 BTN1, SW2 BTN2, SW3 RESET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

Commit message: Connect memory to processor
Parts:
- removed U3: 23lcv1024, Housings_SOIC:SOIC-8_3.9x4.9mm_Pitch1.27mm, symbol 23lcv1024
- added U?: 23lcv1024, symbol modular:23lcv1024
Connections:
- net labels added: SPI1_MISO, SPI1_MOSI, SPI1_SCK
- wire segments 127 -> 167
- no-connect marks 4 -> 5
Changed lines of the file:
@@
-EESchema Schematic File Version 2
+EESchema Schematic File Version 4
 LIBS:modular-rescue
 LIBS:power
 LIBS:device
-LIBS:switches
-LIBS:relays
-LIBS:motors
-LIBS:transistors
-LIBS:conn
-LIBS:linear
-LIBS:regul
 LIBS:74xx
-LIBS:cmos4000
-LIBS:adc-dac
-LIBS:memory
-LIBS:xilinx
-LIBS:microcontrollers
-LIBS:dsp
-LIBS:microchip
-LIBS:analog_switches
-LIBS:motorola
-LIBS:texas
-LIBS:intel
 LIBS:audio
 LIBS:interface
-LIBS:digital-audio
-LIBS:philips
-LIBS:display
-LIBS:cypress
-LIBS:siliconi
-LIBS:opto
-LIBS:atmel
-LIBS:contrib
-LIBS:valves
 LIBS:MCU_ST_STM32
 LIBS:modular
 LIBS:modular-cache
-EELAYER 25 0
+EELAYER 26 0
 EELAYER END
 $Descr A1 33110 23386
@@
 	15950 9200 15950 9300
 Wire Wire Line
-	15950 9300 16250 9300
+	15950 9300 16050 9300
 Wire Wire Line
 	16250 9300 16250 9200
@@
 	15950 5600 15950 5500
 Wire Wire Line
-	15950 5500 16250 5500
+	15950 5500 16050 5500
 Wire Wire Line
 	16250 5500 16250 5600
@@
 	2750 5200 3850 5200
 Wire Wire Line
-	2750 5100 3450 5100
-Wire Wire Line
-	3450 5100 3450 5400
+	2750 5100 3200 5100
+Wire Wire Line
+	3450 5100 3450 5300
 Wire Wire Line
 	3450 5300 3550 5300
@@
 	3200 5700 3200 5800
 Wire Wire Line
-	3200 5800 3450 5800
+	3200 5800 3300 5800
 Wire Wire Line
 	3450 5800 3450 5700
@@
 	4250 5750 4150 5750
 Wire Wire Line
-	4150 5750 4150 5950
+	4150 5750 4150 5850
 Wire Wire Line
 	4150 5950 4250 5950
 Wire Wire Line
-	3950 5850 4250 5850
+	3950 5850 4150 5850
 Connection ~ 4150 5850
 Wire Wire Line
-	3950 5750 3950 6100
+	3950 5750 3950 5850
 Wire Wire Line
 	4950 6500 4950 6400
 Wire Wire Line
-	3950 6500 4950 6500
+	3950 6500 4850 6500
 Wire Wire Line
 	4850 6500 4850 6400
 Wire Wire Line
-	3950 6400 3950 6600
+	3950 6400 3950 6500
 Connection ~ 4850 6500
 Connection ~ 3950 6500
@@
 	2900 4900 2900 4800
 Wire Wire Line
-	2900 4500 2900 4300
+	2900 4500 2900 4400
 Wire Wire Line
 	2900 4000 2900 3900
@@
 	4100 3550 4100 3450
 Wire Wire Line
-	3900 3450 4600 3450
+	3900 3450 4100 3450
 Wire Wire Line
 	4600 3450 4600 3550
@@
 	4100 3850 4100 3950
 Wire Wire Line
-	3900 3950 4600 3950
+	3900 3950 4100 3950
 Wire Wire Line
 	4600 3950 4600 3850
@@
 	6350 4000 6350 3900
 Wire Wire Line
-	6350 3900 6700 3900
+	6350 3900 6550 3900
 Wire Wire Line
 	6700 3900 6700 4000
@@
 	7100 10050 7100 10150
 Wire Wire Line
-	6300 10050 6500 10050
+	6300 10050 6400 10050
 Text Label 6400 9850 0    60   ~ 0
 BTN1
@@
 	7100 10800 7100 10900
 Wire Wire Line
-	6300 10800 6500 10800
+	6300 10800 6400 10800
 Text Label 6400 10600 0    60   ~ 0
 BTN2
@@
 $EndComp
 Wire Wire Line
-	9350 6200 10650 6200
+	9350 6200 9550 6200
 Wire Wire Line
 	9550 6200 9550 6300
@@
 	9850 5100 9850 4950
 Wire Wire Line
-	9850 4950 10350 4950
+	9850 4950 10100 4950
 Wire Wire Line
 	10350 4950 10350 5050
@@
 	10350 5450 10350 5550
 Wire Wire Line
-	10350 5550 9850 5550
+	10350 5550 10100 5550
 Wire Wire Line
 	9850 5550 9850 5400
@@
 Connection ~ 10100 5550
 $Comp
-L 23lcv1024 U3
-U 1 1 5BD6EECB
-P 13650 11700
-F 0 "U3" H 13400 12000 60  0000 C CNN
-F 1 "23lcv1024" H 13750 11400 60  0000 C CNN
-F 2 "Housings_SOIC:SOIC-8_3.9x4.9mm_Pitch1.27mm" H 13650 11700 60  0001 C CNN
-F 3 "" H 13650 11700 60  0001 C CNN
-	1    13650 11700
-	1    0    0    -1
-$EndComp
-$Comp
 L +3V3 #PWR?
 U 1 1 5BD730D3
-P 14500 11400
-F 0 "#PWR?" H 14500 11250 50  0001 C CNN
-F 1 "+3V3" H 14500 11540 50  0000 C CNN
-F 2 "" H 14500 11400 50  0001 C CNN
-F 3 "" H 14500 11400 50  0001 C CNN
-	1    14500 11400
+P 15850 10250
+F 0 "#PWR?" H 15850 10100 50  0001 C CNN
+F 1 "+3V3" H 15850 10390 50  0000 C CNN
+F 2 "" H 15850 10250 50  0001 C CNN
+F 3 "" H 15850 10250 50  0001 C CNN
+	1    15850 10250
 	1    0    0    -1
 $EndComp
@@
 L GND #PWR?
 U 1 1 5BD73159
-P 13000 12050
-F 0 "#PWR?" H 13000 11800 50  0001 C CNN
-F 1 "GND" H 13000 11900 50  0000 C CNN
-F 2 "" H 13000 12050 50  0001 C CNN
-F 3 "" H 13000 12050 50  0001 C CNN
-	1    13000 12050
-	1    0    0    -1
-$EndComp
+P 13400 10300
+F 0 "#PWR?" H 13400 10050 50  0001 C CNN
+F 1 "GND" H 13400 10150 50  0000 C CNN
+F 2 "" H 13400 10300 50  0001 C CNN
+F 3 "" H 13400 10300 50  0001 C CNN
+	1    13400 10300
+	-1   0    0    1
+$EndComp
+Wire Wire Line
+	16150 9300 16250 9300
+Wire Wire Line
+	16050 9300 16100 9300
+Wire Wire Line
+	16100 9300 16150 9300
+Wire Wire Line
+	16150 5500 16250 5500
+Wire Wire Line
+	16050 5500 16100 5500
+Wire Wire Line
+	16100 5500 16150 5500
+Wire Wire Line
+	3200 5100 3450 5100
+Wire Wire Line
+	3450 5300 3450 5400
+Wire Wire Line
+	3300 5800 3450 5800
+Wire Wire Line
+	4150 5850 4150 5950
+Wire Wire Line
+	4150 5850 4250 5850
+Wire Wire Line
+	4850 6500 4950 6500
+Wire Wire Line
+	3950 6500 3950 6600
+Wire Wire Line
+	2900 4400 2900 4300
+Wire Wire Line
+	4350 3450 4600 3450
+Wire Wire Line
+	4350 3950 4600 3950
+Wire Wire Line
+	4100 3450 4350 3450
+Wire Wire Line
+	4100 3950 4350 3950
+Wire Wire Line
+	3950 5850 3950 6100
+Wire Wire Line
+	6550 3900 6700 3900
+Wire Wire Line
+	6400 10050 6500 10050
+Wire Wire Line
+	6400 10800 6500 10800
+Wire Wire Line
+	9550 6200 10650 6200
+Wire Wire Line
+	10100 4950 10350 4950
+Wire Wire Line
+	10100 5550 9850 5550
+$Comp
+L modular:23lcv1024 U?
+U 1 1 5BEA6D78
+P 14300 10500
+F 0 "U?" H 14375 10937 60  0000 C CNN
+F 1 "23lcv1024" H 14375 10831 60  0000 C CNN
+F 2 "" H 14300 10500 60  0001 C CNN
+F 3 "" H 14300 10500 60  0001 C CNN
+	1    14300 10500
+	1    0    0    -1
+$EndComp
+Wire Wire Line
+	13400 10300 13600 10300
+Wire Wire Line
+	13800 10300 13800 10350
+Wire Wire Line
+	13800 10650 13600 10650
+Wire Wire Line
+	13600 10650 13600 10300
+Connection ~ 13600 10300
+Wire Wire Line
+	13600 10300 13800 10300
+Wire Wire Line
+	14950 10350 15850 10350
+Wire Wire Line
+	15850 10350 15850 10250
+NoConn ~ 13800 10550
+$Comp
+L GND #PWR?
+U 1 1 5BECEB98
+P 15900 11100
+F 0 "#PWR?" H 15900 10850 50  0001 C CNN
+F 1 "GND" H 15900 10950 50  0000 C CNN
+F 2 "" H 15900 11100 50  0001 C CNN
+F 3 "" H 15900 11100 50  0001 C CNN
+	1    15900 11100
+	1    0    0    -1
+$EndComp
+Wire Wire Line
+	14950 10450 15900 10450
+Wire Wire Line
+	15900 10450 15900 11100
+Text Label 15150 10550 0    50   ~ 0
+SPI1_SCK
+Text Label 15150 10650 0    50   ~ 0
+SPI1_MOSI
+Text Label 13350 10450 2    50   ~ 0
+SPI1_MISO
+Text Label 10300 7600 2    50   ~ 0
+SPI1_SCK
+Text Label 10300 7800 2    50   ~ 0
+SPI1_MOSI
+Text Label 10300 7700 2    50   ~ 0
+SPI1_MISO
+Wire Wire Line
+	14950 10550 15150 10550
+Wire Wire Line
+	14950 10650 15150 10650
+Wire Wire Line
+	10300 7800 10650 7800
+Wire Wire Line
+	10300 7700 10650 7700
+Wire Wire Line
+	10300 7600 10650 7600
+Wire Wire Line
+	13350 10450 13800 10450
 $EndSCHEMATC

Commit message: Connect DACs and ADCs
Parts:
- C1, C2, C3, C4, C5, C6, C7, C8: symbol C -> modular-rescue:C-
- D1, D2, D3, D4, D5, D6: symbol LED -> modular-rescue:LED-
- J1: symbol USB_OTG -> modular-rescue:USB_OTG-
- J2, J3, J5, J6: symbol Conn_01x03 -> modular-rescue:Conn_01x03-
- J4: symbol Conn_02x08_Counter_Clockwise -> modular-rescue:Conn_02x08_Counter_Clockwise-
- J7: symbol Conn_01x02 -> modular-rescue:Conn_01x02-
- R1, R10, R11, R12, R13, R2, R3, R4, R5, R6, R7, R8, R9: symbol R -> modular-rescue:R-
- RV1: symbol POT -> modular-rescue:POT-
- SW1, SW2, SW3: symbol SW_Push -> modular-rescue:SW_Push-
- U1: symbol FT230XS-R -> modular-rescue:FT230XS-R-
- U2: symbol STM32F302CCTx -> modular-rescue:STM32F302CCTx-
Connections:
- net labels added: OUTPUT
- net labels removed: OUTPUT1, OUTPUT2
- wire segments 167 -> 170
